Commit message: Add files via upload

File: ur10e.urdf (robot description, URDF)
Before this commit: robot ur, 13 links, 12 joints
Links:
- link base_link_inertia: geometry collision mesh filename=https://https://raw.githubusercontent.com/UniversalRobots/U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; visual mesh filename=https://https://raw.githubusercontent.com/UniversalRobots/U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
- link forearm_link: geometry collision mesh filename=https://https://raw.githubusercontent.com/UniversalRobots/U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; visual mesh filename=https://https://raw.githubusercontent.com/UniversalRobots/U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
- link shoulder_link: geometry collision mesh filename=https://https://raw.githubusercontent.com/UniversalRobots/U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; visual mesh filename=https://https://raw.githubusercontent.com/UniversalRobots/U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
- link upper_arm_link: geometry collision mesh filename=https://https://raw.githubusercontent.com/UniversalRobots/U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; visual mesh filename=https://https://raw.githubusercontent.com/UniversalRobots/U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
- link wrist_1_link: geometry collision mesh filename=https://https://raw.githubusercontent.com/UniversalRobots/U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; visual mesh filename=https://https://raw.githubusercontent.com/UniversalRobots/U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
- link wrist_2_link: geometry collision mesh filename=https://https://raw.githubusercontent.com/UniversalRobots/U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; visual mesh filename=https://https://raw.githubusercontent.com/UniversalRobots/U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
- link wrist_3_link: geometry collision mesh filename=https://https://raw.githubusercontent.com/UniversalRobots/U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; visual mesh filename=https://https://raw.githubusercontent.com/UniversalRobots/U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

Commit message: Add files via upload

File: ur10e.urdf (robot description, URDF)
Before this commit: robot ur, 13 links, 12 joints
Links:
- link base_link_inertia: geometry collision mesh filename=https://raw.githubusercontent.com/UniversalRobots/Universal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; visual mesh filename=https://raw.githubusercontent.com/UniversalRobots/Universal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
- link forearm_link: geometry collision mesh filename=https://raw.githubusercontent.com/UniversalRobots/Universal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; visual mesh filename=https://raw.githubusercontent.com/UniversalRobots/Universal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
- link shoulder_link: geometry collision mesh filename=https://raw.githubusercontent.com/UniversalRobots/Universal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; visual mesh filename=https://raw.githubusercontent.com/UniversalRobots/Universal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
- link upper_arm_link: geometry collision mesh filename=https://raw.githubusercontent.com/UniversalRobots/Universal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; visual mesh filename=https://raw.githubusercontent.com/UniversalRobots/Universal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
- link wrist_1_link: geometry collision mesh filename=https://raw.githubusercontent.com/UniversalRobots/Universal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; visual mesh filename=https://raw.githubusercontent.com/UniversalRobots/Universal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
- link wrist_2_link: geometry collision mesh filename=https://raw.githubusercontent.com/UniversalRobots/Universal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; visual mesh filename=https://raw.githubusercontent.com/UniversalRobots/Universal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
- link wrist_3_link: geometry collision mesh filename=https://raw.githubusercontent.com/UniversalRobots/Universal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; visual mesh filename=https://raw.githubusercontent.com/UniversalRobots/Universal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
